Commit message: Prepare force torque state controller

File: ur_robot_driver/resources/ur5_system_position_only.ros2_control.xacro (robot description, xacro)
@@ -43,5 +43,5 @@
         <state_interface name="velocity"/>
         <state_interface name="effort"/>
-      </joint>
+      </joint>tcp_
       <joint name="wrist_2_joint">
         <command_interface name="position">
