Commit message: Remove hardcoded parameters for driver components.

File: ur_ros2_control_demos/urdf/ur5.urdf.xacro (robot description, xacro)
@@ -1,4 +1,8 @@
 <?xml version="1.0"?>
 <robot name="ur5" xmlns:xacro="http://wiki.ros.org/xacro">
+  <xacro:arg name="script_filename" default="$(find ur_robot_driver)/resources/ros_control.urscript"/>
+  <xacro:arg name="output_recipe_filename" default="$(find ur_robot_driver)/resources/rtde_output_recipe.txt"/>
+  <xacro:arg name="input_recipe_filename" default="$(find ur_robot_driver)/resources/rtde_input_recipe.txt"/>
+  <xacro:arg name="robot_ip" default="10.0.1.186"/>
   <link name="base_link" >
     <visual>
@@ -187,4 +191,10 @@
  <!-- Import ur5 ros2_control description -->
  <xacro:include filename="ur5_system_position_only.ros2_control.xacro" />
- <xacro:ur5_system_position_only name="URPositionHardwareInterface" prefix="" />
+ <xacro:ur5_system_position_only name="URPositionHardwareInterface" prefix=""
+                                 script_filename="$(arg script_filename)"
+                                 output_recipe_filename="$(arg output_recipe_filename)"
+                                 input_recipe_filename="$(arg input_recipe_filename)"
+                                 tf_prefix=""
+                                 hash_kinematics=""
+                                 robot_ip="$(arg robot_ip)" />
 </robot>

File: ur_ros2_control_demos/urdf/ur5_system_position_only.ros2_control.xacro (robot description, xacro)
@@ -1,23 +1,23 @@
 <?xml version="1.0"?>
 <robot xmlns:xacro="http://www.ros.org/wiki/xacro">
-  <xacro:macro name="ur5_system_position_only" params="name prefix">
+  <xacro:macro name="ur5_system_position_only" params="name prefix script_filename output_recipe_filename input_recipe_filename tf_prefix hash_kinematics robot_ip">
     <ros2_control name="${name}" type="system">
       <hardware>
         <plugin>ur_robot_driver/URPositionHardwareInterface</plugin>
-        <param name="ramp_time">1.0</param> <!-- ramp time in seconds defining the joint speed by 180/ramp_time [deg/s] -->
+        <param name="ramp_time">5.0</param> <!-- ramp time in seconds defining the joint speed by 180/ramp_time [deg/s] -->
         <param name="rate">600.0</param> <!-- same rate as in controller_manager:ros__parameters:update_rate: 2  -->
-        <param name="robot_ip">10.0.1.186</param>
-        <param name="script_filename">/home/abishalini/ws_ur5e/src/Universal_Robots_ROS2_Driver/ur_robot_driver/resources/ros_control.urscript</param>
-        <param name="output_recipe_filename">/home/abishalini/ws_ur5e/src/Universal_Robots_ROS2_Driver/ur_robot_driver/resources/rtde_output_recipe.txt</param>
-        <param name="input_recipe_filename">/home/abishalini/ws_ur5e/src/Universal_Robots_ROS2_Driver/ur_robot_driver/resources/rtde_input_recipe.txt</param>
+        <param name="robot_ip">${robot_ip}</param>
+        <param name="script_filename">${script_filename}</param>
+        <param name="output_recipe_filename">${output_recipe_filename}</param>
+        <param name="input_recipe_filename">${input_recipe_filename}</param>
         <param name="headless_mode">0</param>
         <param name="reverse_port">50001</param>
         <param name="script_sender_port">50002</param>
-        <param name="tf_prefix">'</param>
+        <param name="tf_prefix">"${tf_prefix}"</param>
         <param name="non_blocking_read">0</param>
         <param name="servoj_gain">2000</param>
         <param name="servoj_lookahead_time">0.03</param>
         <param name="use_tool_communication">0</param>
-        <param name="kinematics/hash">'</param>
+        <param name="kinematics/hash">"${hash_kinematics}"</param>
         <param name="tool_voltage">0</param>
         <param name="tool_parity">0</param>
