Commit message: Move all urdf files to one package.

File: ur_ros2_control_demos/urdf/ur5_system_position_only.ros2_control.xacro (robot description, xacro)
@@ -1,5 +1,8 @@
 <?xml version="1.0"?>
 <robot xmlns:xacro="http://www.ros.org/wiki/xacro">
-  <xacro:macro name="ur5_system_position_only" params="name prefix script_filename output_recipe_filename input_recipe_filename tf_prefix hash_kinematics robot_ip">
+  <xacro:macro name="ur5_system_position_only" params="name prefix
+    script_filename output_recipe_filename
+    input_recipe_filename tf_prefix
+    hash_kinematics robot_ip">
     <ros2_control name="${name}" type="system">
       <hardware>
